File: ReactionGameBoard/reactionGameBoard.kicad_sch (KiCad schematic)
At the start: 15 parts, among them J3 Conn_02x03_Counter_Clockwise, SW1 SW_Push, SW2 SW_DPDT_x2, U1 ATtiny24A-SS, U2 74HC595

Commit message: new board design + code
Parts:
- removed J3: Conn_02x03_Counter_Clockwise, Connector_PinHeader_2.54mm:PinHeader_2x03_P2.54mm_Vertical, symbol Connector_Generic:Conn_02x03_Counter_Clockwise
- added J1, J10, J2, J3, J5, J6, J9: Conn_01x01_Pin, Connector_PinHeader_2.54mm:PinHeader_1x01_P2.54mm_Vertical, symbol Connector:Conn_01x01_Pin
Connections:
- net +3V0: now also J10.1 (Pin_1)
- net A: now also R8.2; no longer R3.2
- net C: now also R2.2; no longer R5.2
- net D: now also R6.2; no longer R7.2
- net DP1: now also U1.12 (PA1); no longer U1.11 (PA2)
- net DP2: now also U1.13 (AREF/PA0); no longer U1.10 (PA3)
- net DP3: now also U1.5 (PB2); no longer U1.6 (PA7)
- net DP4: now also U1.11 (PA2); no longer U1.12 (PA1)
- net Dp: now also R4.2; no longer R6.2
- net E: now also R5.2; no longer R8.2
- net F: now also R7.2; no longer R2.2
- net G: now also R3.2; no longer R4.2
- net GND: now also J9.1 (Pin_1)
- net MISO: now also J2.1 (Pin_1)
- net MOSI: now also U2.14 (SER), J1.1 (Pin_1)
- net SCK: now also U2.11 (SRCLK), J6.1 (Pin_1)
- net reset: now also J5.1 (Pin_1)
- net PA0 renamed PB2
- net PB2: now also U1.3 (XTAL2/PB1); no longer U1.13 (AREF/PA0)
- net clock renamed serialCS
- net serialCS: now also J3.1 (Pin_1); no longer U2.11 (SRCLK)
- removed net data: U1.5 (PB2), U2.14 (SER)
- net latch renamed CS2
- net CS2: now also U1.10 (PA3); no longer U1.3 (XTAL2/PB1)
- no-connect marks 2 -> 3

Commit message: cnc pcb version
Connections:
- net A: now also R1.2; no longer R8.2
- net B: now also R4.2; no longer R1.2
- net C: now also R7.2; no longer R2.2
- net D: now also R3.2; no longer R6.2
- net DP1: now also DS1.9 (2); no longer DS1.12 (1)
- net DP2: now also DS1.12 (1); no longer DS1.9 (2)
- net DP3: now also U1.11 (PA2); no longer U1.5 (PB2)
- net DP4: now also U1.5 (PB2); no longer U1.11 (PA2)
- net Dp: now also R8.2; no longer R4.2
- net E: now also R2.2; no longer R5.2
- net F: now also R5.2; no longer R7.2
- net G: now also R6.2; no longer R3.2
Other:
- moved on the sheet: DS1, U2
